File: splitflap-pcb/splitflap-pcb.sch (KiCad schematic (older format))
At the start: 16 parts, among them J1 INPUT CONN, J2 HALL 1, J3 HALL 2, J4 STEPPER 1, J5 STEPPER 2, J6 OUTPUT CONN, J7 AVR-ISP-6, U1 REGULATOR, U2 ATtiny88-AU, U3 TPIC6595

Commit message: Redesign PCB, connectors are too big
Parts:
- J1, J6: footprint Connector_PinHeader_2.54mm:PinHeader_1x04_P2.54mm_Vertical -> Connector_JST:JST_XH_B4B-XH-AM_1x04_P2.50mm_Vertical
- J2, J3: footprint Connector_PinHeader_2.54mm:PinHeader_1x03_P2.54mm_Vertical -> Connector_JST:JST_XH_B3B-XH-AM_1x03_P2.50mm_Vertical
- J4, J5: footprint Connector_PinHeader_2.54mm:PinHeader_1x05_P2.54mm_Vertical -> Connector_JST:JST_XH_B5B-XH-AM_1x05_P2.50mm_Vertical
Changed lines of the file:
@@
 F 0 "J4" V 3496 3048 50  0000 L CNN
 F 1 "STEPPER 1" V 3587 3048 50  0000 L CNN
-F 2 "Connector_PinHeader_2.54mm:PinHeader_1x05_P2.54mm_Vertical" H 3650 2800 50  0001 C CNN
+F 2 "Connector_JST:JST_XH_B5B-XH-AM_1x05_P2.50mm_Vertical" H 3650 2800 50  0001 C CNN
 F 3 "~" H 3650 2800 50  0001 C CNN
 	1    3650 2800
@@
 F 0 "J5" V 4596 3048 50  0000 L CNN
 F 1 "STEPPER 2" V 4687 3048 50  0000 L CNN
-F 2 "Connector_PinHeader_2.54mm:PinHeader_1x05_P2.54mm_Vertical" H 4750 2800 50  0001 C CNN
+F 2 "Connector_JST:JST_XH_B5B-XH-AM_1x05_P2.50mm_Vertical" H 4750 2800 50  0001 C CNN
 F 3 "~" H 4750 2800 50  0001 C CNN
 	1    4750 2800
@@
 F 0 "J2" V 3238 3112 50  0000 R CNN
 F 1 "HALL 1" V 3150 3100 50  0000 R CNN
-F 2 "Connector_PinHeader_2.54mm:PinHeader_1x03_P2.54mm_Vertical" H 3300 3300 50  0001 C CNN
+F 2 "Connector_JST:JST_XH_B3B-XH-AM_1x03_P2.50mm_Vertical" H 3300 3300 50  0001 C CNN
 F 3 "~" H 3300 3300 50  0001 C CNN
 	1    3300 3300
@@
 F 0 "J3" V 4088 3112 50  0000 R CNN
 F 1 "HALL 2" V 3997 3112 50  0000 R CNN
-F 2 "Connector_PinHeader_2.54mm:PinHeader_1x03_P2.54mm_Vertical" H 4150 3300 50  0001 C CNN
+F 2 "Connector_JST:JST_XH_B3B-XH-AM_1x03_P2.50mm_Vertical" H 4150 3300 50  0001 C CNN
 F 3 "~" H 4150 3300 50  0001 C CNN
 	1    4150 3300
@@
 F 0 "J6" H 6128 2026 50  0000 L CNN
 F 1 "OUTPUT CONN" H 6128 1935 50  0000 L CNN
-F 2 "Connector_PinHeader_2.54mm:PinHeader_1x04_P2.54mm_Vertical" H 6100 2050 50  0001 C CNN
+F 2 "Connector_JST:JST_XH_B4B-XH-AM_1x04_P2.50mm_Vertical" H 6100 2050 50  0001 C CNN
 F 3 "~" H 6100 2050 50  0001 C CNN
 	1    6100 2050
@@
 F 0 "J1" H 1128 2476 50  0000 L CNN
 F 1 "INPUT CONN" H 1128 2385 50  0000 L CNN
-F 2 "Connector_PinHeader_2.54mm:PinHeader_1x04_P2.54mm_Vertical" H 1100 2500 50  0001 C CNN
+F 2 "Connector_JST:JST_XH_B4B-XH-AM_1x04_P2.50mm_Vertical" H 1100 2500 50  0001 C CNN
 F 3 "~" H 1100 2500 50  0001 C CNN
 	1    1100 2500

Commit message: Actually the correct footprints
Parts:
- U1: footprint Package_TO_SOT_SMD:TO-252-3_TabPin2 -> Package_TO_SOT_SMD:TO-252-2
Changed lines of the file:
@@
 F 0 "U1" H 1300 3550 50  0000 C CNN
 F 1 "REGULATOR" H 1300 3450 50  0000 C CNN
-F 2 "Package_TO_SOT_SMD:TO-252-3_TabPin2" H 1300 3400 50  0001 C CNN
+F 2 "Package_TO_SOT_SMD:TO-252-2" H 1300 3400 50  0001 C CNN
 F 3 "http://www.advanced-monolithic.com/pdf/ds1117.pdf" H 1400 2950 50  0001 C CNN
 	1    1300 3200

Commit message: placed components
Parts:
- J1, J6: footprint Connector_JST:JST_XH_B4B-XH-AM_1x04_P2.50mm_Vertical -> Connector_JST:JST_XH_B4B-XH-A_1x04_P2.50mm_Vertical
- J2, J3: footprint Connector_JST:JST_XH_B3B-XH-AM_1x03_P2.50mm_Vertical -> Connector_JST:JST_XH_B3B-XH-A_1x03_P2.50mm_Vertical
- J4, J5: footprint Connector_JST:JST_XH_B5B-XH-AM_1x05_P2.50mm_Vertical -> Connector_JST:JST_XH_B5B-XH-A_1x05_P2.50mm_Vertical
Connections:
- net +12V: now also J6.4 (Pin_4); no longer J6.1 (Pin_1)
- net GND: now also J6.3 (Pin_3); no longer J6.2 (Pin_2)
- net SCL: now also J6.2 (Pin_2); no longer J6.3 (Pin_3)
- net SDA: now also J6.1 (Pin_1); no longer J6.4 (Pin_4)
- net at U3.14 (DRAIN4): now also J4.4 (Pin_4); no longer J4.1 (Pin_1)
- net at U3.15 (DRAIN5): now also J4.3 (Pin_3); no longer J4.2 (Pin_2)
- net at U3.16 (DRAIN6): now also J4.2 (Pin_2); no longer J4.3 (Pin_3)
- net at U3.17 (DRAIN7): now also J4.1 (Pin_1); no longer J4.4 (Pin_4)
Changed lines of the file:
@@
 F 0 "J4" V 3496 3048 50  0000 L CNN
 F 1 "STEPPER 1" V 3587 3048 50  0000 L CNN
-F 2 "Connector_JST:JST_XH_B5B-XH-AM_1x05_P2.50mm_Vertical" H 3650 2800 50  0001 C CNN
+F 2 "Connector_JST:JST_XH_B5B-XH-A_1x05_P2.50mm_Vertical" H 3650 2800 50  0001 C CNN
 F 3 "~" H 3650 2800 50  0001 C CNN
 	1    3650 2800
@@
 F 0 "J5" V 4596 3048 50  0000 L CNN
 F 1 "STEPPER 2" V 4687 3048 50  0000 L CNN
-F 2 "Connector_JST:JST_XH_B5B-XH-AM_1x05_P2.50mm_Vertical" H 4750 2800 50  0001 C CNN
+F 2 "Connector_JST:JST_XH_B5B-XH-A_1x05_P2.50mm_Vertical" H 4750 2800 50  0001 C CNN
 F 3 "~" H 4750 2800 50  0001 C CNN
 	1    4750 2800
@@
 F 0 "J2" V 3238 3112 50  0000 R CNN
 F 1 "HALL 1" V 3150 3100 50  0000 R CNN
-F 2 "Connector_JST:JST_XH_B3B-XH-AM_1x03_P2.50mm_Vertical" H 3300 3300 50  0001 C CNN
+F 2 "Connector_JST:JST_XH_B3B-XH-A_1x03_P2.50mm_Vertical" H 3300 3300 50  0001 C CNN
 F 3 "~" H 3300 3300 50  0001 C CNN
 	1    3300 3300
@@
 F 0 "J3" V 4088 3112 50  0000 R CNN
 F 1 "HALL 2" V 3997 3112 50  0000 R CNN
-F 2 "Connector_JST:JST_XH_B3B-XH-AM_1x03_P2.50mm_Vertical" H 4150 3300 50  0001 C CNN
+F 2 "Connector_JST:JST_XH_B3B-XH-A_1x03_P2.50mm_Vertical" H 4150 3300 50  0001 C CNN
 F 3 "~" H 4150 3300 50  0001 C CNN
 	1    4150 3300
@@
 F 0 "J6" H 6128 2026 50  0000 L CNN
 F 1 "OUTPUT CONN" H 6128 1935 50  0000 L CNN
-F 2 "Connector_JST:JST_XH_B4B-XH-AM_1x04_P2.50mm_Vertical" H 6100 2050 50  0001 C CNN
+F 2 "Connector_JST:JST_XH_B4B-XH-A_1x04_P2.50mm_Vertical" H 6100 2050 50  0001 C CNN
 F 3 "~" H 6100 2050 50  0001 C CNN
 	1    6100 2050
@@
 F 0 "J1" H 1128 2476 50  0000 L CNN
 F 1 "INPUT CONN" H 1128 2385 50  0000 L CNN
-F 2 "Connector_JST:JST_XH_B4B-XH-AM_1x04_P2.50mm_Vertical" H 1100 2500 50  0001 C CNN
+F 2 "Connector_JST:JST_XH_B4B-XH-A_1x04_P2.50mm_Vertical" H 1100 2500 50  0001 C CNN
 F 3 "~" H 1100 2500 50  0001 C CNN
 	1    1100 2500
@@
 Text GLabel 1750 2600 2    50   BiDi ~ 0
 SDA
-Text GLabel 5900 2150 0    50   BiDi ~ 0
+Text GLabel 5900 2050 0    50   BiDi ~ 0
 SCL
-Text GLabel 5900 2250 0    50   BiDi ~ 0
+Text GLabel 5900 1950 0    50   BiDi ~ 0
 SDA
 $Comp
@@
 $EndComp
 $Comp
-L power:+12V #PWR017
-U 1 1 5CC3A7A0
-P 5900 1950
-F 0 "#PWR017" H 5900 1800 50  0001 C CNN
-F 1 "+12V" V 5915 2078 50  0000 L CNN
-F 2 "" H 5900 1950 50  0001 C CNN
-F 3 "" H 5900 1950 50  0001 C CNN
-	1    5900 1950
-	0    -1   -1   0
-$EndComp
-$Comp
 L power:GND #PWR018
 U 1 1 5CC3AAE8
-P 5900 2050
-F 0 "#PWR018" H 5900 1800 50  0001 C CNN
-F 1 "GND" V 5905 1922 50  0000 R CNN
-F 2 "" H 5900 2050 50  0001 C CNN
-F 3 "" H 5900 2050 50  0001 C CNN
-	1    5900 2050
-	0    1    1    0
+P 5550 2150
+F 0 "#PWR018" H 5550 1900 50  0001 C CNN
+F 1 "GND" H 5500 2050 50  0000 R CNN
+F 2 "" H 5550 2150 50  0001 C CNN
+F 3 "" H 5550 2150 50  0001 C CNN
+	1    5550 2150
+	1    0    0    -1
 $EndComp
 $Comp
@@
 	1    0    0    -1
 $EndComp
-Wire Wire Line
-	3550 2600 3550 2300
-Wire Wire Line
-	3550 2300 4100 2300
-Wire Wire Line
-	4100 2300 4100 2050
-Wire Wire Line
-	3650 2600 3650 2350
-Wire Wire Line
-	3650 2350 4200 2350
-Wire Wire Line
-	4200 2350 4200 2050
-Wire Wire Line
-	3750 2600 3750 2400
-Wire Wire Line
-	3750 2400 4300 2400
-Wire Wire Line
-	4300 2400 4300 2050
-Wire Wire Line
-	3850 2600 3850 2450
-Wire Wire Line
-	3850 2450 4400 2450
-Wire Wire Line
-	4400 2450 4400 2050
 Wire Wire Line
 	4650 2600 4650 2450
@@
 Wire Wire Line
 	1300 2600 1750 2600
+Wire Wire Line
+	4100 2050 4100 2200
+Wire Wire Line
+	4100 2200 3850 2200
+Wire Wire Line
+	3850 2200 3850 2600
+Wire Wire Line
+	4200 2050 4200 2250
+Wire Wire Line
+	4200 2250 3750 2250
+Wire Wire Line
+	3750 2250 3750 2600
+Wire Wire Line
+	4300 2050 4300 2300
+Wire Wire Line
+	4300 2300 3650 2300
+Wire Wire Line
+	3650 2300 3650 2600
+Wire Wire Line
+	4400 2050 4400 2350
+Wire Wire Line
+	4400 2350 3550 2350
+Wire Wire Line
+	3550 2350 3550 2600
+$Comp
+L power:+12V #PWR017
+U 1 1 5CC3A7A0
+P 5700 2350
+F 0 "#PWR017" H 5700 2200 50  0001 C CNN
+F 1 "+12V" H 5600 2300 50  0000 L CNN
+F 2 "" H 5700 2350 50  0001 C CNN
+F 3 "" H 5700 2350 50  0001 C CNN
+	1    5700 2350
+	1    0    0    -1
+$EndComp
+Wire Wire Line
+	5900 2250 5800 2250
+Wire Wire Line
+	5800 2250 5800 2350
+Wire Wire Line
+	5800 2350 5700 2350
+Wire Wire Line
+	5900 2150 5550 2150
 $EndSCHEMATC

Commit message: Wired
Parts:
- added C4: 0.1uF, Capacitor_SMD:C_0603_1608Metric, symbol Device:C
Connections:
- net +5V: now also C4.2
- net GND: now also C4.1
Changed lines of the file:
@@
 Wire Wire Line
 	5900 2150 5550 2150
+$Comp
+L Device:C C4
+U 1 1 5CC9DB17
+P 5100 1700
+F 0 "C4" V 4848 1700 50  0000 C CNN
+F 1 "0.1uF" V 4939 1700 50  0000 C CNN
+F 2 "Capacitor_SMD:C_0603_1608Metric" H 5138 1550 50  0001 C CNN
+F 3 "~" H 5100 1700 50  0001 C CNN
+	1    5100 1700
+	-1   0    0    1
+$EndComp
+Connection ~ 5100 1550
+$Comp
+L power:GND #PWR03
+U 1 1 5CC9F58A
+P 5100 1850
+F 0 "#PWR03" H 5100 1600 50  0001 C CNN
+F 1 "GND" H 5105 1677 50  0000 C CNN
+F 2 "" H 5100 1850 50  0001 C CNN
+F 3 "" H 5100 1850 50  0001 C CNN
+	1    5100 1850
+	1    0    0    -1
+$EndComp
 $EndSCHEMATC

Commit message: Closer, working on stitching
Parts:
- added H1, H2, H3, H4: MountingHole_Pad, MountingHole:MountingHole_3.2mm_M3_Pad, symbol Mechanical:MountingHole_Pad
- J1, J6: footprint Connector_JST:JST_XH_B4B-XH-A_1x04_P2.50mm_Vertical -> splitflap-pcb:TE_640456-4
- J2, J3: footprint Connector_JST:JST_XH_B3B-XH-A_1x03_P2.50mm_Vertical -> splitflap-pcb:TE_640456-3
Connections:
- net GND: now also H1.1, H2.1, H3.1, H4.1
Other:
- moved on the sheet: J2, J3
Changed lines of the file:
@@
 L Connector:Conn_01x03_Female J2
 U 1 1 5CC1B5A0
-P 3300 3300
-F 0 "J2" V 3238 3112 50  0000 R CNN
-F 1 "HALL 1" V 3150 3100 50  0000 R CNN
-F 2 "Connector_JST:JST_XH_B3B-XH-A_1x03_P2.50mm_Vertical" H 3300 3300 50  0001 C CNN
-F 3 "~" H 3300 3300 50  0001 C CNN
-	1    3300 3300
-	0    -1   -1   0
-$EndComp
-$Comp
-L Connector:Conn_01x03_Female J3
-U 1 1 5CC1C3FA
-P 4150 3300
-F 0 "J3" V 4088 3112 50  0000 R CNN
-F 1 "HALL 2" V 3997 3112 50  0000 R CNN
-F 2 "Connector_JST:JST_XH_B3B-XH-A_1x03_P2.50mm_Vertical" H 4150 3300 50  0001 C CNN
-F 3 "~" H 4150 3300 50  0001 C CNN
-	1    4150 3300
-	0    -1   -1   0
+P 3650 3300
+F 0 "J2" H 3800 3200 50  0000 R CNN
+F 1 "HALL 1" H 3950 3300 50  0000 R CNN
+F 2 "splitflap-pcb:TE_640456-3" H 3650 3300 50  0001 C CNN
+F 3 "~" H 3650 3300 50  0001 C CNN
+	1    3650 3300
+	1    0    0    -1
 $EndComp
 $Comp
@@
 F 0 "J6" H 6128 2026 50  0000 L CNN
 F 1 "OUTPUT CONN" H 6128 1935 50  0000 L CNN
-F 2 "Connector_JST:JST_XH_B4B-XH-A_1x04_P2.50mm_Vertical" H 6100 2050 50  0001 C CNN
+F 2 "splitflap-pcb:TE_640456-4" H 6100 2050 50  0001 C CNN
 F 3 "~" H 6100 2050 50  0001 C CNN
 	1    6100 2050
@@
 F 0 "J1" H 1128 2476 50  0000 L CNN
 F 1 "INPUT CONN" H 1128 2385 50  0000 L CNN
-F 2 "Connector_JST:JST_XH_B4B-XH-A_1x04_P2.50mm_Vertical" H 1100 2500 50  0001 C CNN
+F 2 "splitflap-pcb:TE_640456-4" H 1100 2500 50  0001 C CNN
 F 3 "~" H 1100 2500 50  0001 C CNN
 	1    1100 2500
@@
 L power:+5V #PWR07
 U 1 1 5CC5E099
-P 3050 3500
-F 0 "#PWR07" H 3050 3350 50  0001 C CNN
-F 1 "+5V" H 3065 3673 50  0000 C CNN
-F 2 "" H 3050 3500 50  0001 C CNN
-F 3 "" H 3050 3500 50  0001 C CNN
-	1    3050 3500
+P 3450 3200
+F 0 "#PWR07" H 3450 3050 50  0001 C CNN
+F 1 "+5V" H 3465 3373 50  0000 C CNN
+F 2 "" H 3450 3200 50  0001 C CNN
+F 3 "" H 3450 3200 50  0001 C CNN
+	1    3450 3200
 	1    0    0    -1
 $EndComp
@@
 L power:+5V #PWR09
 U 1 1 5CC5E37F
-P 3900 3500
-F 0 "#PWR09" H 3900 3350 50  0001 C CNN
-F 1 "+5V" H 3915 3673 50  0000 C CNN
-F 2 "" H 3900 3500 50  0001 C CNN
-F 3 "" H 3900 3500 50  0001 C CNN
-	1    3900 3500
-	1    0    0    -1
-$EndComp
-Wire Wire Line
-	4050 3500 3900 3500
-Wire Wire Line
-	3200 3500 3050 3500
+P 4300 3200
+F 0 "#PWR09" H 4300 3050 50  0001 C CNN
+F 1 "+5V" H 4315 3373 50  0000 C CNN
+F 2 "" H 4300 3200 50  0001 C CNN
+F 3 "" H 4300 3200 50  0001 C CNN
+	1    4300 3200
+	1    0    0    -1
+$EndComp
 $Comp
 L power:GND #PWR08
 U 1 1 5CC5F590
-P 3300 3500
-F 0 "#PWR08" H 3300 3250 50  0001 C CNN
-F 1 "GND" H 3305 3327 50  0000 C CNN
-F 2 "" H 3300 3500 50  0001 C CNN
-F 3 "" H 3300 3500 50  0001 C CNN
-	1    3300 3500
+P 3250 3300
+F 0 "#PWR08" H 3250 3050 50  0001 C CNN
+F 1 "GND" H 3255 3127 50  0000 C CNN
+F 2 "" H 3250 3300 50  0001 C CNN
+F 3 "" H 3250 3300 50  0001 C CNN
+	1    3250 3300
 	1    0    0    -1
 $EndComp
@@
 L power:GND #PWR010
 U 1 1 5CC5F89E
-P 4150 3500
-F 0 "#PWR010" H 4150 3250 50  0001 C CNN
-F 1 "GND" H 4155 3327 50  0000 C CNN
-F 2 "" H 4150 3500 50  0001 C CNN
-F 3 "" H 4150 3500 50  0001 C CNN
-	1    4150 3500
+P 4150 3300
+F 0 "#PWR010" H 4150 3050 50  0001 C CNN
+F 1 "GND" H 4155 3127 50  0000 C CNN
+F 2 "" H 4150 3300 50  0001 C CNN
+F 3 "" H 4150 3300 50  0001 C CNN
+	1    4150 3300
 	1    0    0    -1
 $EndComp
@@
 	3650 4250 3650 3900
 Wire Wire Line
-	3650 3900 3400 3900
-Wire Wire Line
-	3400 3900 3400 3500
-Wire Wire Line
 	3750 4250 3750 3900
 Wire Wire Line
 	3750 3900 4250 3900
-Wire Wire Line
-	4250 3900 4250 3500
 Text GLabel 4800 1050 1    50   Input ~ 0
 MOSI
@@
 	1    0    0    -1
 $EndComp
+$Comp
+L Connector:Conn_01x03_Female J3
+U 1 1 5CC1C3FA
+P 4500 3300
+F 0 "J3" H 4700 3200 50  0000 R CNN
+F 1 "HALL 2" H 4800 3300 50  0000 R CNN
+F 2 "splitflap-pcb:TE_640456-3" H 4500 3300 50  0001 C CNN
+F 3 "~" H 4500 3300 50  0001 C CNN
+	1    4500 3300
+	1    0    0    -1
+$EndComp
+Wire Wire Line
+	4300 3300 4150 3300
+Wire Wire Line
+	4250 3400 4300 3400
+Wire Wire Line
+	4250 3400 4250 3900
+Wire Wire Line
+	3450 3300 3250 3300
+Wire Wire Line
+	3650 3900 3450 3900
+Wire Wire Line
+	3450 3900 3450 3400
+$Comp
+L Mechanical:MountingHole_Pad H1
+U 1 1 5CC9621F
+P 1050 6200
+F 0 "H1" H 1150 6249 50  0000 L CNN
+F 1 "MountingHole_Pad" H 1150 6158 50  0000 L CNN
+F 2 "MountingHole:MountingHole_3.2mm_M3_Pad" H 1050 6200 50  0001 C CNN
+F 3 "~" H 1050 6200 50  0001 C CNN
+	1    1050 6200
+	1    0    0    -1
+$EndComp
+$Comp
+L Mechanical:MountingHole_Pad H2
+U 1 1 5CC965B3
+P 1900 6200
+F 0 "H2" H 2000 6249 50  0000 L CNN
+F 1 "MountingHole_Pad" H 2000 6158 50  0000 L CNN
+F 2 "MountingHole:MountingHole_3.2mm_M3_Pad" H 1900 6200 50  0001 C CNN
+F 3 "~" H 1900 6200 50  0001 C CNN
+	1    1900 6200
+	1    0    0    -1
+$EndComp
+$Comp
+L Mechanical:MountingHole_Pad H3
+U 1 1 5CC96C1B
+P 2750 6200
+F 0 "H3" H 2850 6249 50  0000 L CNN
+F 1 "MountingHole_Pad" H 2850 6158 50  0000 L CNN
+F 2 "MountingHole:MountingHole_3.2mm_M3_Pad" H 2750 6200 50  0001 C CNN
+F 3 "~" H 2750 6200 50  0001 C CNN
+	1    2750 6200
+	1    0    0    -1
+$EndComp
+$Comp
+L Mechanical:MountingHole_Pad H4
+U 1 1 5CC978F8
+P 3600 6200
+F 0 "H4" H 3700 6249 50  0000 L CNN
+F 1 "MountingHole_Pad" H 3700 6158 50  0000 L CNN
+F 2 "MountingHole:MountingHole_3.2mm_M3_Pad" H 3600 6200 50  0001 C CNN
+F 3 "~" H 3600 6200 50  0001 C CNN
+	1    3600 6200
+	1    0    0    -1
+$EndComp
+$Comp
+L power:GND #PWR0103
+U 1 1 5CC9844E
+P 3600 6300
+F 0 "#PWR0103" H 3600 6050 50  0001 C CNN
+F 1 "GND" H 3605 6127 50  0000 C CNN
+F 2 "" H 3600 6300 50  0001 C CNN
+F 3 "" H 3600 6300 50  0001 C CNN
+	1    3600 6300
+	1    0    0    -1
+$EndComp
+$Comp
+L power:GND #PWR0104
+U 1 1 5CC98833
+P 2750 6300
+F 0 "#PWR0104" H 2750 6050 50  0001 C CNN
+F 1 "GND" H 2755 6127 50  0000 C CNN
+F 2 "" H 2750 6300 50  0001 C CNN
+F 3 "" H 2750 6300 50  0001 C CNN
+	1    2750 6300
+	1    0    0    -1
+$EndComp
+$Comp
+L power:GND #PWR0105
+U 1 1 5CC98C2E
+P 1900 6300
+F 0 "#PWR0105" H 1900 6050 50  0001 C CNN
+F 1 "GND" H 1905 6127 50  0000 C CNN
+F 2 "" H 1900 6300 50  0001 C CNN
+F 3 "" H 1900 6300 50  0001 C CNN
+	1    1900 6300
+	1    0    0    -1
+$EndComp
+$Comp
+L power:GND #PWR0106
+U 1 1 5CC99018
+P 1050 6300
+F 0 "#PWR0106" H 1050 6050 50  0001 C CNN
+F 1 "GND" H 1055 6127 50  0000 C CNN
+F 2 "" H 1050 6300 50  0001 C CNN
+F 3 "" H 1050 6300 50  0001 C CNN
+	1    1050 6300
+	1    0    0    -1
+$EndComp

Commit message: new netlist
Parts:
- added C5, C6: 0.1uF, Capacitor_SMD:C_0603_1608Metric, symbol Device:C
Connections:
- net +5V: now also C4.1, R3.1, C5.2, C6.1; no longer C4.2, R3.2
- net GND: now also C4.2, C5.1, C6.2; no longer C4.1
- net SCL: now also R2.1; no longer R3.1
- net SDA: now also R3.2; no longer R2.1
- net HALL2SIG: now reaches J3.3 (Pin_3), U2.1 (PD3)
- net HALL1SIG: now reaches J2.3 (Pin_3), U2.32 (PD2)
Other:
- note added: "Hall Effect Sensors"
- note added: "Mounting Holes"
- note added: "i2c pullups"
- moved on the sheet: C1, C2, C3, C4, H1, H2, H3, H4, J1, J2, J3, J4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

Commit message: More
Connections:
- net SCL: now also R3.2; no longer R2.1
- net SDA: now also R2.1; no longer R3.2
Other:
- moved on the sheet: R2, R3
Changed lines of the file:
@@
 $EndComp
 $Comp
-L Device:R R2
-U 1 1 5CC6D9CB
+L Device:R R3
+U 1 1 5CC6DB71
 P 6050 1800
-F 0 "R2" H 6100 1750 50  0000 L CNN
-F 1 "4K7" H 6100 1850 50  0000 L CNN
+F 0 "R3" H 5900 1850 50  0000 L CNN
+F 1 "4K7" H 5850 1750 50  0000 L CNN
 F 2 "Resistor_SMD:R_0603_1608Metric" V 5980 1800 50  0001 C CNN
 F 3 "~" H 6050 1800 50  0001 C CNN
 	1    6050 1800
-	-1   0    0    1
-$EndComp
-$Comp
-L Device:R R3
-U 1 1 5CC6DB71
-P 6150 1800
-F 0 "R3" H 6200 1850 50  0000 L CNN
-F 1 "4K7" H 6200 1750 50  0000 L CNN
-F 2 "Resistor_SMD:R_0603_1608Metric" V 6080 1800 50  0001 C CNN
-F 3 "~" H 6150 1800 50  0001 C CNN
-	1    6150 1800
 	1    0    0    -1
 $EndComp
@@
 Wire Wire Line
 	7250 2900 7250 3100
+$Comp
+L Device:R R2
+U 1 1 5CC6D9CB
+P 6150 1800
+F 0 "R2" H 6000 1750 50  0000 L CNN
+F 1 "4K7" H 5950 1850 50  0000 L CNN
+F 2 "Resistor_SMD:R_0603_1608Metric" V 6080 1800 50  0001 C CNN
+F 3 "~" H 6150 1800 50  0001 C CNN
+	1    6150 1800
+	-1   0    0    1
+$EndComp
 $EndSCHEMATC
