File: splitflap-pcb/splitflap-pcb.sch (KiCad schematic (older format))
At the start: 23 parts, among them J1 INPUT CONN, J2 HALL 1, J3 HALL 2, J4 STEPPER 1, J5 STEPPER 2, J6 OUTPUT CONN, J7 AVR-ISP-6, U1 REGULATOR, U2 ATtiny88-AU, U3 TPIC6595

Commit message: Tweaks
Parts:
- C2: value 0.1uF -> 0.33uF
- U1: value REGULATOR -> NCV78M05
Other:
- note added: "Hall Effect Sensor Connectors"
- note added: "i2c Pull-ups"
- note removed: "Hall Effect Sensors"
- note removed: "i2c pullups"
- moved on the sheet: C1, C5, R1
Changed lines of the file:
@@
 U 1 1 5CC18283
 P 8500 4450
-F 0 "J4" V 8346 4698 50  0000 L CNN
-F 1 "STEPPER 1" V 8437 4698 50  0000 L CNN
+F 0 "J4" V 8700 4400 50  0000 L CNN
+F 1 "STEPPER 1" V 8600 4250 50  0000 L CNN
 F 2 "Connector_JST:JST_XH_B5B-XH-A_1x05_P2.50mm_Vertical" H 8500 4450 50  0001 C CNN
 F 3 "~" H 8500 4450 50  0001 C CNN
@@
 U 1 1 5CC19C75
 P 8500 3350
-F 0 "J5" V 8346 3598 50  0000 L CNN
-F 1 "STEPPER 2" V 8437 3598 50  0000 L CNN
+F 0 "J5" V 8700 3300 50  0000 L CNN
+F 1 "STEPPER 2" V 8600 3150 50  0000 L CNN
 F 2 "Connector_JST:JST_XH_B5B-XH-A_1x05_P2.50mm_Vertical" H 8500 3350 50  0001 C CNN
 F 3 "~" H 8500 3350 50  0001 C CNN
@@
 P 3700 3250
 F 0 "C2" H 3500 3300 50  0000 L CNN
-F 1 "0.1uF" H 3350 3200 50  0000 L CNN
+F 1 "0.33uF" H 3350 3200 50  0000 L CNN
 F 2 "Capacitor_SMD:C_0603_1608Metric" H 3738 3100 50  0001 C CNN
 F 3 "~" H 3700 3250 50  0001 C CNN
@@
 U 1 1 5CC15B7D
 P 3900 1900
-F 0 "J1" V 4150 1800 50  0000 L CNN
+F 0 "J1" V 4100 1850 50  0000 L CNN
 F 1 "INPUT CONN" V 4000 1650 50  0000 L CNN
 F 2 "splitflap-pcb:TE_640456-4" H 3900 1900 50  0001 C CNN
@@
 L power:+5V #PWR06
 U 1 1 5CC391F4
-P 4350 3100
-F 0 "#PWR06" H 4350 2950 50  0001 C CNN
-F 1 "+5V" H 4365 3273 50  0000 C CNN
-F 2 "" H 4350 3100 50  0001 C CNN
-F 3 "" H 4350 3100 50  0001 C CNN
-	1    4350 3100
+P 4400 3100
+F 0 "#PWR06" H 4400 2950 50  0001 C CNN
+F 1 "+5V" H 4415 3273 50  0000 C CNN
+F 2 "" H 4400 3100 50  0001 C CNN
+F 3 "" H 4400 3100 50  0001 C CNN
+	1    4400 3100
 	1    0    0    -1
 $EndComp
@@
 L power:+12V #PWR04
 U 1 1 5CC394D0
-P 3750 3100
-F 0 "#PWR04" H 3750 2950 50  0001 C CNN
-F 1 "+12V" H 3765 3273 50  0000 C CNN
-F 2 "" H 3750 3100 50  0001 C CNN
-F 3 "" H 3750 3100 50  0001 C CNN
-	1    3750 3100
+P 3700 3100
+F 0 "#PWR04" H 3700 2950 50  0001 C CNN
+F 1 "+12V" H 3715 3273 50  0000 C CNN
+F 2 "" H 3700 3100 50  0001 C CNN
+F 3 "" H 3700 3100 50  0001 C CNN
+	1    3700 3100
 	1    0    0    -1
 $EndComp
@@
 Text GLabel 6750 3800 0    50   Input ~ 0
 SS
-Connection ~ 2300 1550
 Text GLabel 2900 2850 2    50   BiDi ~ 0
 SCK
@@
 Text GLabel 2900 2550 2    50   Output ~ 0
 SS
-Wire Wire Line
-	2300 1400 2300 1550
 $Comp
 L power:+5V #PWR01
 U 1 1 5CC3C620
-P 2300 1400
-F 0 "#PWR01" H 2300 1250 50  0001 C CNN
-F 1 "+5V" H 2315 1573 50  0000 C CNN
-F 2 "" H 2300 1400 50  0001 C CNN
-F 3 "" H 2300 1400 50  0001 C CNN
-	1    2300 1400
+P 2300 1300
+F 0 "#PWR01" H 2300 1150 50  0001 C CNN
+F 1 "+5V" H 2315 1473 50  0000 C CNN
+F 2 "" H 2300 1300 50  0001 C CNN
+F 3 "" H 2300 1300 50  0001 C CNN
+	1    2300 1300
 	1    0    0    -1
 $EndComp
@@
 L power:GND #PWR011
 U 1 1 5CC38022
-P 2300 5250
-F 0 "#PWR011" H 2300 5000 50  0001 C CNN
-F 1 "GND" H 2305 5077 50  0000 C CNN
-F 2 "" H 2300 5250 50  0001 C CNN
-F 3 "" H 2300 5250 50  0001 C CNN
-	1    2300 5250
+P 2300 5150
+F 0 "#PWR011" H 2300 4900 50  0001 C CNN
+F 1 "GND" H 2305 4977 50  0000 C CNN
+F 2 "" H 2300 5150 50  0001 C CNN
+F 3 "" H 2300 5150 50  0001 C CNN
+	1    2300 5150
 	1    0    0    -1
 $EndComp
@@
 P 4050 3100
 F 0 "U1" H 4050 3450 50  0000 C CNN
-F 1 "REGULATOR" H 4050 3350 50  0000 C CNN
+F 1 "NCV78M05" H 4050 3350 50  0000 C CNN
 F 2 "Package_TO_SOT_SMD:TO-252-2" H 4050 3300 50  0001 C CNN
 F 3 "http://www.advanced-monolithic.com/pdf/ds1117.pdf" H 4150 2850 50  0001 C CNN
@@
 Text GLabel 6750 3300 0    50   Input ~ 0
 MOSI
-Connection ~ 3750 3100
 Connection ~ 4050 3400
 $Comp
@@
 $EndComp
 Wire Wire Line
-	3750 3100 3700 3100
-Wire Wire Line
 	3700 3400 4050 3400
 Wire Wire Line
 	4050 3400 4400 3400
-Wire Wire Line
-	4400 3100 4350 3100
-Connection ~ 4350 3100
 $Comp
 L Device:C C1
 U 1 1 5CC6F529
-P 2150 1400
-F 0 "C1" V 2300 1600 50  0000 C CNN
-F 1 "0.1uF" V 2200 1550 50  0000 C CNN
-F 2 "Capacitor_SMD:C_0603_1608Metric" H 2188 1250 50  0001 C CNN
-F 3 "~" H 2150 1400 50  0001 C CNN
-	1    2150 1400
-	0    -1   -1   0
-$EndComp
-Wire Wire Line
-	2300 1550 2000 1550
-Wire Wire Line
-	2300 5250 2300 5150
+P 2450 1300
+F 0 "C1" V 2300 1450 50  0000 C CNN
+F 1 "0.1uF" V 2400 1450 50  0000 C CNN
+F 2 "Capacitor_SMD:C_0603_1608Metric" H 2488 1150 50  0001 C CNN
+F 3 "~" H 2450 1300 50  0001 C CNN
+	1    2450 1300
+	0    1    1    0
+$EndComp
 $Comp
 L Connector:AVR-ISP-6 J7
 U 1 1 5CC7779B
 P 5600 3250
-F 0 "J7" H 5321 3346 50  0000 R CNN
-F 1 "AVR-ISP-6" H 5321 3255 50  0000 R CNN
+F 0 "J7" H 5850 3750 50  0000 R CNN
+F 1 "AVR-ISP-6" H 6000 3650 50  0000 R CNN
 F 2 "Connector_PinHeader_2.54mm:PinHeader_2x03_P2.54mm_Vertical" V 5350 3300 50  0001 C CNN
 F 3 " ~" H 4325 2700 50  0001 C CNN
@@
 Text GLabel 2900 2750 2    50   BiDi ~ 0
 MISO
-Text GLabel 3000 3850 3    50   Input ~ 0
+Text GLabel 3000 3850 2    50   Input ~ 0
 RST
 $Comp
@@
 L power:GND #PWR0101
 U 1 1 5CC88AAA
-P 4400 1750
-F 0 "#PWR0101" H 4400 1500 50  0001 C CNN
-F 1 "GND" H 4500 1750 50  0000 C CNN
-F 2 "" H 4400 1750 50  0001 C CNN
-F 3 "" H 4400 1750 50  0001 C CNN
-	1    4400 1750
+P 4400 1800
+F 0 "#PWR0101" H 4400 1550 50  0001 C CNN
+F 1 "GND" H 4500 1800 50  0000 C CNN
+F 2 "" H 4400 1800 50  0001 C CNN
+F 3 "" H 4400 1800 50  0001 C CNN
+	1    4400 1800
 	1    0    0    -1
 $EndComp
@@
 L power:PWR_FLAG #FLG0102
 U 1 1 5CC8CDF8
-P 4400 1750
-F 0 "#FLG0102" H 4400 1825 50  0001 C CNN
-F 1 "PWR_FLAG" H 4650 1850 50  0001 C CNN
-F 2 "" H 4400 1750 50  0001 C CNN
-F 3 "~" H 4400 1750 50  0001 C CNN
-	1    4400 1750
+P 4400 1800
+F 0 "#FLG0102" H 4400 1875 50  0001 C CNN
+F 1 "PWR_FLAG" H 4650 1900 50  0001 C CNN
+F 2 "" H 4400 1800 50  0001 C CNN
+F 3 "~" H 4400 1800 50  0001 C CNN
+	1    4400 1800
 	1    0    0    -1
 $EndComp
@@
 L Device:R R1
 U 1 1 5CC48A9E
-P 3200 3850
-F 0 "R1" V 2993 3850 50  0000 C CNN
-F 1 "10K" V 3084 3850 50  0000 C CNN
-F 2 "Resistor_SMD:R_0603_1608Metric" V 3130 3850 50  0001 C CNN
-F 3 "~" H 3200 3850 50  0001 C CNN
-	1    3200 3850
+P 3150 3950
+F 0 "R1" V 2943 3950 50  0000 C CNN
+F 1 "10K" V 3034 3950 50  0000 C CNN
+F 2 "Resistor_SMD:R_0603_1608Metric" V 3080 3950 50  0001 C CNN
+F 3 "~" H 3150 3950 50  0001 C CNN
+	1    3150 3950
 	0    -1   -1   0
 $EndComp
@@
 L power:+5V #PWR0102
 U 1 1 5CC49F93
-P 3350 3850
-F 0 "#PWR0102" H 3350 3700 50  0001 C CNN
-F 1 "+5V" H 3365 4023 50  0000 C CNN
-F 2 "" H 3350 3850 50  0001 C CNN
-F 3 "" H 3350 3850 50  0001 C CNN
-	1    3350 3850
+P 3300 3950
+F 0 "#PWR0102" H 3300 3800 50  0001 C CNN
+F 1 "+5V" H 3315 4123 50  0000 C CNN
+F 2 "" H 3300 3950 50  0001 C CNN
+F 3 "" H 3300 3950 50  0001 C CNN
+	1    3300 3950
 	1    0    0    -1
 $EndComp
@@
 L Device:C C5
 U 1 1 5CCA00F0
-P 1850 1550
-F 0 "C5" V 1900 1450 50  0000 C CNN
-F 1 "0.1uF" V 1800 1400 50  0000 C CNN
-F 2 "Capacitor_SMD:C_0603_1608Metric" H 1888 1400 50  0001 C CNN
-F 3 "~" H 1850 1550 50  0001 C CNN
-	1    1850 1550
-	0    -1   -1   0
+P 2600 1450
+F 0 "C5" V 2550 1600 50  0000 C CNN
+F 1 "0.1uF" V 2650 1600 50  0000 C CNN
+F 2 "Capacitor_SMD:C_0603_1608Metric" H 2638 1300 50  0001 C CNN
+F 3 "~" H 2600 1450 50  0001 C CNN
+	1    2600 1450
+	0    1    1    0
 $EndComp
 $Comp
@@
 Wire Wire Line
 	4050 3400 4050 3500
-Connection ~ 2300 1400
-Wire Wire Line
-	1700 1550 1650 1550
-Wire Wire Line
-	2000 1400 1650 1400
-Wire Wire Line
-	1650 1400 1650 1550
 $Comp
 L power:GND #PWR?
 U 1 1 5CCC3192
-P 1650 1550
-F 0 "#PWR?" H 1650 1300 50  0001 C CNN
-F 1 "GND" H 1655 1377 50  0000 C CNN
-F 2 "" H 1650 1550 50  0001 C CNN
-F 3 "" H 1650 1550 50  0001 C CNN
-	1    1650 1550
+P 2950 1450
+F 0 "#PWR?" H 2950 1200 50  0001 C CNN
+F 1 "GND" H 2955 1277 50  0000 C CNN
+F 2 "" H 2950 1450 50  0001 C CNN
+F 3 "" H 2950 1450 50  0001 C CNN
+	1    2950 1450
 	1    0    0    -1
 $EndComp
@@
 Text GLabel 7300 1950 2    50   Output ~ 0
 HALL1SIG
-Text GLabel 2900 4350 0    50   Input ~ 0
+Text GLabel 2900 4350 2    50   Input ~ 0
 HALL1SIG
-Text GLabel 2900 4450 0    50   Input ~ 0
+Text GLabel 2900 4450 2    50   Input ~ 0
 HALL2SIG
 $Comp
@@
 U 1 1 5CC10A0D
 P 2300 3350
-F 0 "U2" V 1600 3300 50  0000 R CNN
-F 1 "ATtiny88-AU" V 1700 3300 50  0000 R CNN
+F 0 "U2" H 2200 3700 50  0000 R CNN
+F 1 "ATtiny88-AU" H 2400 3600 50  0000 R CNN
 F 2 "Package_QFP:TQFP-32_7x7mm_P0.8mm" H 2300 3350 50  0001 C CIN
 F 3 "http://ww1.microchip.com/downloads/en/DeviceDoc/doc8008.pdf" H 2300 3350 50  0001 C CNN
@@
 	1    0    0    -1
 $EndComp
-Wire Wire Line
-	2900 3850 3050 3850
-Connection ~ 1650 1550
 $Comp
 L power:+5V #PWR?
@@
 P 6100 1600
 F 0 "#PWR?" H 6100 1450 50  0001 C CNN
-F 1 "+5V" H 6115 1773 50  0000 C CNN
+F 1 "+5V" H 6200 1700 50  0000 C CNN
 F 2 "" H 6100 1600 50  0001 C CNN
 F 3 "" H 6100 1600 50  0001 C CNN
@@
 	1    0    0    -1
 $EndComp
-Wire Wire Line
-	4100 1800 4200 1800
-Wire Wire Line
-	4200 1800 4200 1750
-Connection ~ 4400 1750
+Connection ~ 4400 1800
 Wire Wire Line
 	4100 1700 4200 1700
@@
 Text Notes 4500 4250 2    50   ~ 0
 Mounting Holes
-Text Notes 6600 1600 2    50   ~ 0
-i2c pullups
-Text Notes 8050 1500 2    50   ~ 0
-Hall Effect Sensors
+Text Notes 6400 1400 2    50   ~ 0
+i2c Pull-ups
+Text Notes 8250 1500 2    50   ~ 0
+Hall Effect Sensor Connectors
 $Comp
 L Mechanical:MountingHole_Pad H1
@@
 	1    0    0    -1
 $EndComp
-Wire Wire Line
-	4200 1750 4400 1750
 Wire Wire Line
 	6950 1950 7100 1950
@@
 	-1   0    0    1
 $EndComp
+Wire Wire Line
+	4350 3100 4400 3100
+Connection ~ 4400 3100
+Wire Wire Line
+	3750 3100 3700 3100
+Connection ~ 3700 3100
+Wire Wire Line
+	4100 1800 4400 1800
+Wire Wire Line
+	2900 3850 3000 3850
+Wire Wire Line
+	3000 3850 3000 3950
+Connection ~ 2300 1550
+Wire Wire Line
+	2300 1300 2300 1450
+Wire Wire Line
+	2300 1450 2450 1450
+Connection ~ 2300 1450
+Wire Wire Line
+	2300 1450 2300 1550
+Wire Wire Line
+	2750 1450 2950 1450
+Wire Wire Line
+	2950 1300 2950 1450
+Wire Wire Line
+	2600 1300 2950 1300
+Connection ~ 2950 1450
+Connection ~ 2300 1300
 $EndSCHEMATC
