File: splitflap-pcb/splitflap-pcb.kicad_pcb (KiCad board)
At the start: 2 copper layers, 50 x 33.3 mm, 23 parts, among them J1 INPUT CONN, J2 HALL 1, J3 HALL 2, J4 STEPPER 1, J5 STEPPER 2, J6 OUTPUT CONN, J7 AVR-ISP-6, U1 REGULATOR, U2 ATtiny88-AU, U3 TPIC6595

Commit message: Tweaks
Parts:
- C2: value 0.1uF -> 0.33uF
- U1: value REGULATOR -> NCV78M05
Routing:
- net GND: vias 194 -> 196
Other:
- board text added: "0.33uF"
- board text added: "TPIC6B595"
- board text removed: "TPIC6595"

Commit message: just before panelizing
Routing:
- net Net-(J4-Pad4): track 6.79 -> 8.36 mm
- net Net-(J4-Pad1): track 7.96 -> 8.63 mm
- net Net-(J4-Pad3): track 6.94 -> 7.61 mm
- net Net-(J4-Pad2): track 7.57 -> 8.12 mm
- net HALL2SIG: track 37.5 -> 38.0 mm
- net GND: vias 196 -> 198
Other:
- board text added: "12V"
- board text added: "GND"
- board text added: "In"
- board text added: "Out"
- board text added: "SCL"
- board text added: "SDA"
- board text added: "SplitFlap S V0.7 2019-05-01 Sam Warmuth"
- board text removed: "12V/I2C"
- board text removed: "SplitFlapI2C V0.6 2019-04-30 Sam Warmuth"

Commit message: v09
Parts:
- added C7: 100uF, Capacitor_THT:CP_Radial_D6.3mm_P2.50mm, F.Cu at (138.3, 118.2)
- moved J7 4.90 mm to (135.4, 127.3), turned to 90 degrees
Routing:
- net RST: track 26.4 -> 17.5 mm
- net +12V: track 83.0 -> 91.5 mm
- net SCK: track 38.0 -> 42.6 mm
- net SCL: track 51.8 -> 55.0 mm, vias 5 -> 3
- net HALL2SIG: track 38.0 -> 35.1 mm
- net MOSI: track 28.5 -> 31.1 mm
- net SDA: track 54.4 -> 56.0 mm
- net HALL1SIG: track 48.1 -> 48.7 mm
- net +5V: track 112.5 -> 112.0 mm
- net GND: vias 198 -> 194
Other:
- board text added: "100uF"
- board text added: "SplitFlap S V0.9 2019-05-02 Sam Warmuth"
- board text removed: "SplitFlap S V0.7 2019-05-01 Sam Warmuth"

Commit message: v10, almost ready to order
Routing:
- net GND: vias 194 -> 191
Other:
- board text added: "SplitFlap S 1.0 2019-05-03 Sam Warmuth"
- board text removed: "SplitFlap S V0.9 2019-05-02 Sam Warmuth"
